File: examples/buck-48v-24v-1kw/kicad/03_gate.kicad_sch (KiCad schematic)
At the start: 16 parts, among them U1 UCC27211DDAR

Commit message: feat: complete six-layer power PCB routing and pass native DRC
Parts:
- U1: footprint Package_SO:SOIC-8-1EP_3.9x4.9mm_P1.27mm_EP2.29x3mm -> Package_SO:SOIC-8-1EP_3.9x4.9mm_P1.27mm_EP2.95x4.9mm_Mask2.71x3.4mm
Changed lines of the file:
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@@
           (property "Reference" "U1" (at 322.58000000000004 62.23000000000002 0)  (effects (font (size 1.27 1.27))))
 (property "Value" "UCC27211DDAR" (at 322.58000000000004 64.77000000000001 0)  (effects (font (size 1.27 1.27))))
-(property "Footprint" "Package_SO:SOIC-8-1EP_3.9x4.9mm_P1.27mm_EP2.29x3mm" (at 322.58000000000004 76.20000000000002 0) (hide yes) (effects (font (size 1.27 1.27))))
+(property "Footprint" "Package_SO:SOIC-8-1EP_3.9x4.9mm_P1.27mm_EP2.95x4.9mm_Mask2.71x3.4mm" (at 322.58000000000004 76.20000000000002 0) (hide yes) (effects (font (size 1.27 1.27))))
 (property "Datasheet" "" (at 322.58000000000004 76.20000000000002 0) (hide yes) (effects (font (size 1.27 1.27))))
           (pin "1")
