File: examples/buck-48v-24v-1kw/kicad/05_aux5.kicad_sch (KiCad schematic)
At the start: 13 parts, among them U3 TPS54302DDCR

Commit message: feat: complete six-layer power PCB routing and pass native DRC
Other:
- moved on the sheet: C44, C45, L3
Changed lines of the file:
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@@
           (effects (font (size 1.0 1.0)) (justify left))
 )
-(symbol (lib_id "AIPE:Sym_L3") (at 101.6 76.2 0)
+(symbol (lib_id "AIPE:Sym_L3") (at 101.6 81.28 0)
           (unit 1) (in_bom yes) (on_board yes) (dnp no)
           (property "Reference" "L3" (at 101.6 67.31 0)  (effects (font (size 1.27 1.27))))
-(property "Value" "10uH" (at 101.6 69.85000000000001 0)  (effects (font (size 1.27 1.27))))
-(property "Footprint" "Inductor_SMD:L_Coilcraft_MSS1048-XXX" (at 101.6 76.2 0) (hide yes) (effects (font (size 1.27 1.27))))
-(property "Datasheet" "" (at 101.6 76.2 0) (hide yes) (effects (font (size 1.27 1.27))))
+(property "Value" "10uH" (at 101.6 69.85 0)  (effects (font (size 1.27 1.27))))
+(property "Footprint" "Inductor_SMD:L_Coilcraft_MSS1048-XXX" (at 101.6 81.28 0) (hide yes) (effects (font (size 1.27 1.27))))
+(property "Datasheet" "" (at 101.6 81.28 0) (hide yes) (effects (font (size 1.27 1.27))))
           (pin "1")
 (pin "2")
           (instances (project "AIPE_Buck_1kW" (path "/558e48a2-11d7-5e19-b5b7-8bc9de1ba629/b3b20e2d-8d59-5df7-baf2-d5a18e5b34c9"
             (reference "L3") (unit 1)))))
-(wire (pts (xy 93.97999999999999 76.2) (xy 91.44 76.2))
+(wire (pts (xy 101.6 77.47) (xy 99.06 77.47))
           (stroke (width 0) (type default)))
 (global_label "SW5" (shape bidirectional)
-          (at 91.44 76.2 180)
+          (at 99.06 77.47 180)
           (effects (font (size 1.0 1.0)) (justify right))
 )
-(wire (pts (xy 109.22 76.2) (xy 111.76 76.2))
+(wire (pts (xy 101.6 85.09) (xy 99.06 85.09))
           (stroke (width 0) (type default)))
 (global_label "5V" (shape bidirectional)
-          (at 111.76 76.2 0)
-          (effects (font (size 1.0 1.0)) (justify left))
+          (at 99.06 85.09 180)
+          (effects (font (size 1.0 1.0)) (justify right))
 )
 (symbol (lib_id "AIPE:Sym_C42") (at 165.1 76.2 0)
@@
           (effects (font (size 1.0 1.0)) (justify left))
 )
-(symbol (lib_id "AIPE:Sym_C44") (at 38.1 104.14 0)
+(symbol (lib_id "AIPE:Sym_C44") (at 38.1 114.3 0)
           (unit 1) (in_bom yes) (on_board yes) (dnp no)
-          (property "Reference" "C44" (at 38.1 95.25 0)  (effects (font (size 1.27 1.27))))
-(property "Value" "56p/50V" (at 38.1 97.79 0)  (effects (font (size 1.27 1.27))))
-(property "Footprint" "Capacitor_SMD:C_0805_2012Metric" (at 38.1 104.14 0) (hide yes) (effects (font (size 1.27 1.27))))
-(property "Datasheet" "" (at 38.1 104.14 0) (hide yes) (effects (font (size 1.27 1.27))))
+          (property "Reference" "C44" (at 38.1 105.41 0)  (effects (font (size 1.27 1.27))))
+(property "Value" "56p/50V" (at 38.1 107.95 0)  (effects (font (size 1.27 1.27))))
+(property "Footprint" "Capacitor_SMD:C_0805_2012Metric" (at 38.1 114.3 0) (hide yes) (effects (font (size 1.27 1.27))))
+(property "Datasheet" "" (at 38.1 114.3 0) (hide yes) (effects (font (size 1.27 1.27))))
           (pin "1")
 (pin "2")
           (instances (project "AIPE_Buck_1kW" (path "/558e48a2-11d7-5e19-b5b7-8bc9de1ba629/b3b20e2d-8d59-5df7-baf2-d5a18e5b34c9"
             (reference "C44") (unit 1)))))
-(wire (pts (xy 30.48 104.14) (xy 27.94 104.14))
+(wire (pts (xy 30.48 114.3) (xy 27.94 114.3))
           (stroke (width 0) (type default)))
 (global_label "5V" (shape bidirectional)
-          (at 27.94 104.14 180)
+          (at 27.94 114.3 180)
           (effects (font (size 1.0 1.0)) (justify right))
 )
-(wire (pts (xy 45.72 104.14) (xy 48.26 104.14))
+(wire (pts (xy 45.72 114.3) (xy 48.26 114.3))
           (stroke (width 0) (type default)))
 (global_label "FB5" (shape bidirectional)
-          (at 48.26 104.14 0)
+          (at 48.26 114.3 0)
           (effects (font (size 1.0 1.0)) (justify left))
 )
-(symbol (lib_id "AIPE:Sym_C45") (at 101.6 104.14 0)
+(symbol (lib_id "AIPE:Sym_C45") (at 101.6 114.3 0)
           (unit 1) (in_bom yes) (on_board yes) (dnp no)
-          (property "Reference" "C45" (at 101.6 95.25 0)  (effects (font (size 1.27 1.27))))
-(property "Value" "220u/16V" (at 101.6 97.79 0)  (effects (font (size 1.27 1.27))))
-(property "Footprint" "Capacitor_THT:CP_Radial_D6.3mm_P2.50mm" (at 101.6 104.14 0) (hide yes) (effects (font (size 1.27 1.27))))
-(property "Datasheet" "" (at 101.6 104.14 0) (hide yes) (effects (font (size 1.27 1.27))))
+          (property "Reference" "C45" (at 101.6 105.41 0)  (effects (font (size 1.27 1.27))))
+(property "Value" "220u/16V" (at 101.6 107.95 0)  (effects (font (size 1.27 1.27))))
+(property "Footprint" "Capacitor_THT:CP_Radial_D6.3mm_P2.50mm" (at 101.6 114.3 0) (hide yes) (effects (font (size 1.27 1.27))))
+(property "Datasheet" "" (at 101.6 114.3 0) (hide yes) (effects (font (size 1.27 1.27))))
           (pin "1")
 (pin "2")
           (instances (project "AIPE_Buck_1kW" (path "/558e48a2-11d7-5e19-b5b7-8bc9de1ba629/b3b20e2d-8d59-5df7-baf2-d5a18e5b34c9"
             (reference "C45") (unit 1)))))
-(wire (pts (xy 93.97999999999999 104.14) (xy 91.44 104.14))
+(wire (pts (xy 93.97999999999999 114.3) (xy 91.44 114.3))
           (stroke (width 0) (type default)))
 (global_label "5V" (shape bidirectional)
-          (at 91.44 104.14 180)
+          (at 91.44 114.3 180)
           (effects (font (size 1.0 1.0)) (justify right))
 )
-(wire (pts (xy 109.22 104.14) (xy 111.76 104.14))
+(wire (pts (xy 109.22 114.3) (xy 111.76 114.3))
           (stroke (width 0) (type default)))
 (global_label "GND" (shape bidirectional)
-          (at 111.76 104.14 0)
+          (at 111.76 114.3 0)
           (effects (font (size 1.0 1.0)) (justify left))
 )
