File: examples/buck-48v-24v-1kw/kicad/12_clock_debug.kicad_sch (KiCad schematic)
At the start: 20 parts, among them J7 TI 14-pin JTAG; key pin 6 abs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, J8 SCI boot strap; default open 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, J9 UART 3.3 V only, Y1 30MHz/3V3

Commit message: feat: complete six-layer power PCB routing and pass native DRC
Parts:
- J8: value SCI boot strap; default open / Flash -> BOOT: 1-2 SCI / 2-3 or open Flash
Connections:
- net BOOT84: now also J8.2; no longer J8.1
- net GND: now also J8.1; no longer J8.2
Changed lines of the file:
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@@
           (unit 1) (in_bom yes) (on_board yes) (dnp no)
           (property "Reference" "J8" (at 193.04 120.65 0)  (effects (font (size 1.27 1.27))))
-(property "Value" "SCI boot strap; default open / Flash" (at 193.04 123.19 0)  (effects (font (size 1.27 1.27))))
+(property "Value" "BOOT: 1-2 SCI / 2-3 or open Flash" (at 193.04 123.19 0)  (effects (font (size 1.27 1.27))))
 (property "Footprint" "Connector_PinHeader_2.54mm:PinHeader_1x03_P2.54mm_Vertical" (at 193.04 130.81 0) (hide yes) (effects (font (size 1.27 1.27))))
 (property "Datasheet" "" (at 193.04 130.81 0) (hide yes) (effects (font (size 1.27 1.27))))
@@
 (wire (pts (xy 168.91 129.54) (xy 166.37 129.54))
           (stroke (width 0) (type default)))
-(global_label "BOOT84" (shape bidirectional)
+(global_label "GND" (shape bidirectional)
           (at 166.37 129.54 180)
           (effects (font (size 1.0 1.0)) (justify right))
@@
 (wire (pts (xy 168.91 132.08) (xy 166.37 132.08))
           (stroke (width 0) (type default)))
-(global_label "GND" (shape bidirectional)
+(global_label "BOOT84" (shape bidirectional)
           (at 166.37 132.08 180)
           (effects (font (size 1.0 1.0)) (justify right))
