File: examples/sic-buck-400v-200v-5kw/kicad/control_board/02_supplies.kicad_sch (KiCad schematic)
At the start: 35 parts, among them J2 J_RESET: manual reset through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, Q1 MMBT3904,215, U2 TPS54302DDCR, U3 TPS767D301PWPR, U4 TPS3808G01DBVR

Commit message: feat(v2.1): example regenerated - wired schematics, both boards routed with the upgraded router, exports, crops, validation
Schematics (wired style, gates passed): ERC 0 on both projects (power 20261012T075113Z-erc-df18ce6e,
control 20261012T075120Z-erc-7a14cacb); netlist (ref,pad)->net exact vs the model and vs the frozen V2
netlists with equal net names; .kicad_dru / net_settings identical to the legacy generation; stub
global labels 648 -> 7 (power) and 667 -> 7 (control), wired pin share 0 -> 0.90 / 0.76, junctions,
hierarchical labels and power symbols introduced, continuation sheets removed; readability metrics
V2 vs V2.1 in engineering_checks/schematic_readability_*.

Power board (octilinear simplification + tangent arcs on the V2 search; 8-direction search kept
opt-in after attempt A left 2 connections open): 0 unresolved, DRC 0/0/0 (20261012T090308Z-drc-8fd50803),
segments 4755 -> 2991 + 145 arcs, 90-degree bends 3609 -> 1121, stair runs 382 -> 124, length
5744.6 -> 5545.6 mm, vias 606 = V2, no net longer / more vias / narrower. Control board: 0 unresolved,
DRC 0/0/0 (20261012T084327Z-drc-7f07f983), segments 5995 -> 4262 + 261 arcs, 90-degree bends
4069 -> 1233, stair runs 435 -> 144, length 7055.2 -> 6700.7 mm, vias 798 = V2, 96 nets shorter,
0 longer. FOOTPRINT.SetDNP for DNP parts (schematic parity), beautify anchors bound to off-grid vias
by copper overlap (path_geometry.connected_by_overlap), In2.Cu inner pass styled.

Exports 11/11 per board, renders and layer PDFs refreshed, high-resolution V2/V2.1 crops under
review/crops/, routing_quality_* and v21_validation.{json,md} (nine TASK 7 checks independently
re-derived). verify_sic_buck passed; 338 tests OK (2 skipped).

Co-Authored-By: Claude Fable 5.1 <noreply@anthropic.com>
Other:
- note added: "Supply provenance (PWR_FLAG)"
- note added: "TPS3808 5 V supervisor and reset"
- note added: "TPS54302 5 V buck"
- note added: "TPS767D301 dual LDO, core-first sequencing"
- moved on the sheet: D2, J2, L1, Q1, U2, U3, U4
