File: examples/sic-buck-400v-200v-5kw/kicad/control_board/02_supplies.kicad_sch (KiCad schematic)
At the start: 35 parts, among them J2 J_RESET: manual reset through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, Q1 MMBT3904,215, U2 TPS54302DDCR, U3 TPS767D301PWPR, U4 TPS3808G01DBVR

Commit message: Correct sensing circuits and add verified V2.2 local bypasses
Parts:
- added C76: 100n/50V, Capacitor_SMD:C_0603_1608Metric, symbol AIPE:Sym_C76
Connections:
- net 3V3: now also C76.1
- net GND_CTRL: now also C76.2
Other:
- note added: "U4 dedicated local bypass (V2.2)"
- moved on the sheet: C10, C11, C12, C13, C14, C15, C16, C4, C5, C6, C7, C8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
