File: examples/sic-buck-400v-200v-5kw/kicad/control_board/06_pwm_fault_logic.kicad_sch (KiCad schematic)
At the start: 33 parts, among them J6 J_ESTOP: normally-closed E-st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, U10 SN74LV21APWR, U11 SN74LV04APWR, U12 REF3125AIDBZR, U6 SN74LVC2G08DCTR, U7 SN74LVC1G74DCTR, U8 SN74LV21APWR, U9 SN74LV21APWR

Commit message: feat(v2.1): example regenerated - wired schematics, both boards routed with the upgraded router, exports, crops, validation
Schematics (wired style, gates passed): ERC 0 on both projects (power 20261012T075113Z-erc-df18ce6e,
control 20261012T075120Z-erc-7a14cacb); netlist (ref,pad)->net exact vs the model and vs the frozen V2
netlists with equal net names; .kicad_dru / net_settings identical to the legacy generation; stub
global labels 648 -> 7 (power) and 667 -> 7 (control), wired pin share 0 -> 0.90 / 0.76, junctions,
hierarchical labels and power symbols introduced, continuation sheets removed; readability metrics
V2 vs V2.1 in engineering_checks/schematic_readability_*.

Power board (octilinear simplification + tangent arcs on the V2 search; 8-direction search kept
opt-in after attempt A left 2 connections open): 0 unresolved, DRC 0/0/0 (20261012T090308Z-drc-8fd50803),
segments 4755 -> 2991 + 145 arcs, 90-degree bends 3609 -> 1121, stair runs 382 -> 124, length
5744.6 -> 5545.6 mm, vias 606 = V2, no net longer / more vias / narrower. Control board: 0 unresolved,
DRC 0/0/0 (20261012T084327Z-drc-7f07f983), segments 5995 -> 4262 + 261 arcs, 90-degree bends
4069 -> 1233, stair runs 435 -> 144, length 7055.2 -> 6700.7 mm, vias 798 = V2, 96 nets shorter,
0 longer. FOOTPRINT.SetDNP for DNP parts (schematic parity), beautify anchors bound to off-grid vias
by copper overlap (path_geometry.connected_by_overlap), In2.Cu inner pass styled.

Exports 11/11 per board, renders and layer PDFs refreshed, high-resolution V2/V2.1 crops under
review/crops/, routing_quality_* and v21_validation.{json,md} (nine TASK 7 checks independently
re-derived). verify_sic_buck passed; 338 tests OK (2 skipped).

Co-Authored-By: Claude Fable 5.1 <noreply@anthropic.com>
Parts:
- added C54: 100n/50V, Capacitor_SMD:C_0603_1608Metric, symbol AIPE:Sym_C54
- added C55: 100n/50V, Capacitor_SMD:C_0603_1608Metric, symbol AIPE:Sym_C55
- added C56: 100n/50V, Capacitor_SMD:C_0603_1608Metric, symbol AIPE:Sym_C56
- added C57: 100n/50V, Capacitor_SMD:C_0603_1608Metric, symbol AIPE:Sym_C57
- added C58: 100n/50V, Capacitor_SMD:C_0603_1608Metric, symbol AIPE:Sym_C58
- added C59: 100n/50V, Capacitor_SMD:C_0603_1608Metric, symbol AIPE:Sym_C59
- added C60: 100n/50V, Capacitor_SMD:C_0603_1608Metric, symbol AIPE:Sym_C60
- added C61: 100n/50V, Capacitor_SMD:C_0603_1608Metric, symbol AIPE:Sym_C61
- added C62: 100n/50V, Capacitor_SMD:C_0603_1608Metric, symbol AIPE:Sym_C62
- added R59: 21.5k, Resistor_SMD:R_0603_1608Metric, symbol AIPE:Sym_R59
- added R60: 10k, Resistor_SMD:R_0603_1608Metric, symbol AIPE:Sym_R60
- added R61: 10k, Resistor_SMD:R_0603_1608Metric, symbol AIPE:Sym_R61
- added R62: 10k, Resistor_SMD:R_0603_1608Metric, symbol AIPE:Sym_R62
- added R63: 10k, Resistor_SMD:R_0603_1608Metric, symbol AIPE:Sym_R63
- added U13: TLV1702AIDGKR, Package_SO:VSSOP-8_3x3mm_P0.65mm, symbol AIPE:Sym_U13
- added U14: TLV1702AIDGKR, Package_SO:VSSOP-8_3x3mm_P0.65mm, symbol AIPE:Sym_U14
Connections:
- net 3V3: now also C55.1, C56.1, C57.1, C58.1, C59.1, C60.1, C61.1, C62.1, R60.1, R61.1, R62.1, R63.1, U13.8 (V+), U14.8 (V+)
- net GND_CTRL: now also C54.2, C55.2, C56.2, C57.2, C58.2, C59.2, C60.2, C61.2, C62.2, U13.4 (V-), U14.4 (V-)
- net OTP_N: now also R63.2, U14.7 (2OUT)
- net OVP_IN_N: now also R60.2, U13.1 (1OUT)
- net OVP_IN_REF: now also U13.3 (1IN+)
- net OVP_OUT_N: now also R61.2, U13.7 (2OUT)
- net OVP_OUT_REF: now also U13.5 (2IN+)
- net UVLO: now also R59.1, R62.2, U14.1 (1OUT)
- net UVLO_REF: now also C54.1, R59.2, U14.3 (1IN+)
- new net OTP_REF: U14.6 (2IN-)
- new net TEMP_HS_NTC: U14.5 (2IN+)
- new net VIN_SENSE: U13.2 (1IN-), U14.2 (1IN-)
- new net VOUT_SENSE: U13.6 (2IN-)
Other:
- note added: "Fault combiners, polarity restoration, pull-ups, E-stop"
- note added: "Fault latch (SN74LVC1G74)"
- note added: "Logic supply bypass"
- note added: "PWM gating (SN74LVC2G08)"
- note added: "REF3125 reference and OVP / UVLO thresholds"
- note added: "TLV1702 comparators"
- moved on the sheet: J6, U10, U11, U12, U6, U7, U8, U9
