File: examples/sic-buck-400v-200v-5kw/kicad/control_board/06_pwm_fault_logic.kicad_sch (KiCad schematic)
At the start: 49 parts, among them J6 J_ESTOP: normally-closed E-st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, U10 SN74LV21APWR, U11 SN74LV04APWR, U12 REF3125AIDBZR, U13 TLV1702AIDGKR, U14 TLV1702AIDGKR, U6 SN74LVC2G08DCTR, U7 SN74LVC1G74DCTR, U8 SN74LV21APWR, U9 SN74LV21APWR

Commit message: Correct sensing circuits and add verified V2.2 local bypasses
Parts:
- added C77: 100n/50V, Capacitor_SMD:C_0603_1608Metric, symbol AIPE:Sym_C77
- added C78: 100n/50V, Capacitor_SMD:C_0603_1608Metric, symbol AIPE:Sym_C78
- added C79: 100n/50V, Capacitor_SMD:C_0603_1608Metric, symbol AIPE:Sym_C79
Connections:
- net 3V3: now also C77.1, C78.1, C79.1
- net GND_CTRL: now also C77.2, C78.2, C79.2
Other:
- note added: "U10 dedicated local bypass (V2.2)"
- note added: "U11 dedicated local bypass (V2.2)"
- note added: "U8 dedicated local bypass (V2.2)"
- moved on the sheet: C50, C51, C52, C53, C54, C55, C56, C57, C58, C59, C60, C61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
