File: examples/sic-buck-400v-200v-5kw/kicad/control_board/05_clock_debug.kicad_sch (KiCad schematic)
At the start: 17 parts, among them J3 J_JTAG: TI 14-pin, key pin 6 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, J4 J_BOOT: jumper 1-2 = SCI-A bo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, J5 J_UART: SCI-A, 3.3 V levels o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, Y1 ASV-30.000MHZ-EJ-T

Commit message: Correct sensing circuits and add verified V2.2 local bypasses
Other:
- moved on the sheet: C49, J3, J4, J5, R26, R27, R28, R29, R30, R31, R32, R33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
