File: examples/sic-buck-400v-200v-5kw/kicad/control_board/AIPE_SiC_Buck_Control.kicad_pcb (KiCad board)
At the start: 4 copper layers, 120 x 80 mm, 207 parts, among them J1 12 V in, J2 J_RESET: manual reset through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, J3 J_JTAG: TI 14-pin, key pin 6 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, J4 J_BOOT: jumper 1-2 = SCI-A bo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, J5 J_UART: SCI-A, 3.3 V levels o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, J6 J_ESTOP: normally-closed E-st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, J7 J_NTC: Vishay NTCALUG01A103F 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, J8 J_MEZZ: 2 x 25 header to the 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, Q1 MMBT3904,215, U1 TPS26400PWPR, U10 SN74LV21APWR, U11 SN74LV04APWR, U12 REF3125AIDBZR, U13 TLV1702AIDGKR, U14 TLV1702AIDGKR, U15 REF3130AIDBZR, U16 LM61CIM3/NOPB, U2 TPS54302DDCR, U3 TPS767D301PWPR, U4 TPS3808G01DBVR, U5 TMS320F28335PGFA, U6 SN74LVC2G08DCTR, U7 SN74LVC1G74DCTR, U8 SN74LV21APWR, U9 SN74LV21APWR, Y1 ASV-30.000MHZ-EJ-T

Commit message: Correct sensing circuits and add verified V2.2 local bypasses
Parts:
- added C76: 100n/50V, Capacitor_SMD:C_0603_1608Metric, B.Cu at (16.5, 48.5)
- added C77: 100n/50V, Capacitor_SMD:C_0603_1608Metric, B.Cu at (68.8, 57.5)
- added C78: 100n/50V, Capacitor_SMD:C_0603_1608Metric, B.Cu at (54.8, 57.8)
- added C79: 100n/50V, Capacitor_SMD:C_0603_1608Metric, B.Cu at (60.1, 70.5)
Routing:
- net 3V3: track 121.4 -> 131.6 mm, vias 84 -> 87
- net GND_CTRL: track 227.5 -> 231.1 mm, vias 161 -> 165
Other:
- board text added: "AIPE SiC BUCK CONTROL V2.2"
- board text removed: "AIPE SiC BUCK CONTROL V2.1"
