File: examples/sic-buck-400v-200v-5kw/kicad/control_board/AIPE_SiC_Buck_Control.kicad_sch (KiCad schematic)
At the start: 0 parts

Commit message: Correct sensing circuits and add verified V2.2 local bypasses
Other:
- note added: "AI-GENERATED ENGINEERING PROTOTYPE - V2.2 - HUMAN REVIEW REQUIRED"
- note removed: "AI-GENERATED ENGINEERING PROTOTYPE - V2.1 - HUMAN REVIEW REQUIRED"
- title: AIPE V2 SiC buck control board - 400 V (360-440 V) to 200 V / 25 A / 5 kW / 50 kHz synchronous buck; Wolfspeed C4MS025120K; TMS320F28335 control board on a stacked SELV mezzanine -> SiC buck 400V / 200V / 5kW - control board
