File: examples/sic-buck-400v-200v-5kw/kicad/power_board/01_power_stage.kicad_sch (KiCad schematic)
At the start: 42 parts, among them J1 VIN_RAW (+IN), J2 PGND (-IN), J3 VOUT (+OUT), J4 PGND (-OUT), J5 RLY_A (VIN_RAW), J6 RLY_B (VIN), Q1 C4MS025120K, Q2 C4MS025120K, U10 TMCS1133C2AQDVGR

Commit message: feat(v2.1): example regenerated - wired schematics, both boards routed with the upgraded router, exports, crops, validation
Schematics (wired style, gates passed): ERC 0 on both projects (power 20261012T075113Z-erc-df18ce6e,
control 20261012T075120Z-erc-7a14cacb); netlist (ref,pad)->net exact vs the model and vs the frozen V2
netlists with equal net names; .kicad_dru / net_settings identical to the legacy generation; stub
global labels 648 -> 7 (power) and 667 -> 7 (control), wired pin share 0 -> 0.90 / 0.76, junctions,
hierarchical labels and power symbols introduced, continuation sheets removed; readability metrics
V2 vs V2.1 in engineering_checks/schematic_readability_*.

Power board (octilinear simplification + tangent arcs on the V2 search; 8-direction search kept
opt-in after attempt A left 2 connections open): 0 unresolved, DRC 0/0/0 (20261012T090308Z-drc-8fd50803),
segments 4755 -> 2991 + 145 arcs, 90-degree bends 3609 -> 1121, stair runs 382 -> 124, length
5744.6 -> 5545.6 mm, vias 606 = V2, no net longer / more vias / narrower. Control board: 0 unresolved,
DRC 0/0/0 (20261012T084327Z-drc-7f07f983), segments 5995 -> 4262 + 261 arcs, 90-degree bends
4069 -> 1233, stair runs 435 -> 144, length 7055.2 -> 6700.7 mm, vias 798 = V2, 96 nets shorter,
0 longer. FOOTPRINT.SetDNP for DNP parts (schematic parity), beautify anchors bound to off-grid vias
by copper overlap (path_geometry.connected_by_overlap), In2.Cu inner pass styled.

Exports 11/11 per board, renders and layer PDFs refreshed, high-resolution V2/V2.1 crops under
review/crops/, routing_quality_* and v21_validation.{json,md} (nine TASK 7 checks independently
re-derived). verify_sic_buck passed; 338 tests OK (2 skipped).

Co-Authored-By: Claude Fable 5.1 <noreply@anthropic.com>
Parts:
- added C17: 0.47u/630V, Capacitor_SMD:C_2220_5750Metric, symbol AIPE:Sym_C17
- added C18: 10n/300VAC, Capacitor_THT:C_Disc_D12.5mm_W5.0mm_P10.00mm, symbol AIPE:Sym_C18
- added C19: 10n/300VAC, Capacitor_THT:C_Disc_D12.5mm_W5.0mm_P10.00mm, symbol AIPE:Sym_C19
- added H1: PE M4 stud, MountingHole:MountingHole_4.3mm_M4_Pad, symbol AIPE:Sym_H1
- added R13: 0.47, Resistor_SMD:R_2512_6332Metric, symbol AIPE:Sym_R13
- added R14: 0, Resistor_SMD:R_2512_6332Metric, symbol AIPE:Sym_R14
- added R15: 1M, Resistor_SMD:R_2512_6332Metric, symbol AIPE:Sym_R15
- added R16: 1M, Resistor_SMD:R_2512_6332Metric, symbol AIPE:Sym_R16
- C15, C16, R11, R12, RV1: now not fitted
Connections:
- net DAMP_MID: now also C17.2, R13.1
- net PGND: now also C19.1, R13.2, R14.1, R15.1
- net VIN: now also C17.1, C18.1
- new net PE: C18.2, C19.2, H1.1, R14.2, R16.2
- new net PE_REF_MID: R15.2, R16.1
Other:
- note added: "Bleeders and LIVE indicators"
- note added: "Half bridge, HF capacitor bank, DC-link capacitors"
- note added: "Output inductor, current sensor, output capacitors"
- note added: "PE network"
- note added: "Power terminals, precharge PTC, MOV"
- note added: "Snubber and damping leg (DNP)"
- note added: "Supply provenance (PWR_FLAG)"
- moved on the sheet: D1, D2, J1, J2, J3, J4, J5, J6, L1, Q1, Q2, R11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
