File: examples/sic-buck-400v-200v-5kw/kicad/power_board/01_power_stage.kicad_sch (KiCad schematic)
At the start: 50 parts, among them J1 VIN_RAW (+IN), J2 PGND (-IN), J3 VOUT (+OUT), J4 PGND (-OUT), J5 RLY_A (VIN_RAW), J6 RLY_B (VIN), Q1 C4MS025120K, Q2 C4MS025120K, U10 TMCS1133C2AQDVGR

Commit message: Correct sensing circuits and add verified V2.2 local bypasses
Other:
- moved on the sheet: C1, C10, C11, C12, C13, C14, C15, C16, C17, C18, C19, C2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
