File: examples/sic-buck-400v-200v-5kw/kicad/power_board/02_gate_driver_hs.kicad_sch (KiCad schematic)
At the start: 31 parts, among them U1 UCC21710QDWRQ1

Commit message: fix(pcb): structural DRC sources removed at the schematic level; layout review and stage-3 evidence
Power project regenerated (ERC 0 findings, run 20261010T165532Z): UCC21710 drivers now use
an AIPE footprint that carries its own 1.2 x 16.6 mm isolation slot (no library
silkscreen crossing a board cut-out), the AMC1311 slot is lengthened to 10.8 mm, the
LED anode nodes of the indicator strings form a PGND_LV class of the PGND reference
island (0.3 mm to PGND instead of a 3 mm HV spacing an 0805 LED cannot meet), and the
pin-field exceptions now cover no-connect pads whose unconnected-* nets fall into
KiCad's Default class. 45 design rules; nothing weakened.

Also records the independent layout review of the first routed state
(pcb_rule_review.md, 19 findings), the correction pass before/after tables, the
stage-3 power-board routing experiments and patch set, the stage-1 floorplan
generator with its candidate comparison, run_check report hashes and the verifier
hash fix.

Co-Authored-By: Claude Fable 5.1 <noreply@anthropic.com>
Parts:
- U1: footprint Package_SO:SOIC-16W_7.5x10.3mm_P1.27mm -> AIPE:UCC21710_DW0016A_Slot
Changed lines of the file:
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@@
           (property "Reference" "U1" (at 240.03 34.29 0)  (effects (font (size 1.27 1.27))))
 (property "Value" "UCC21710QDWRQ1" (at 240.03 36.83 0)  (effects (font (size 1.27 1.27))))
-(property "Footprint" "Package_SO:SOIC-16W_7.5x10.3mm_P1.27mm" (at 240.03 52.07 0) (hide yes) (effects (font (size 1.27 1.27))))
+(property "Footprint" "AIPE:UCC21710_DW0016A_Slot" (at 240.03 52.07 0) (hide yes) (effects (font (size 1.27 1.27))))
 (property "Datasheet" "" (at 240.03 52.07 0) (hide yes) (effects (font (size 1.27 1.27))))
           (pin "1")

Commit message: feat(v2.1): example regenerated - wired schematics, both boards routed with the upgraded router, exports, crops, validation
Schematics (wired style, gates passed): ERC 0 on both projects (power 20261012T075113Z-erc-df18ce6e,
control 20261012T075120Z-erc-7a14cacb); netlist (ref,pad)->net exact vs the model and vs the frozen V2
netlists with equal net names; .kicad_dru / net_settings identical to the legacy generation; stub
global labels 648 -> 7 (power) and 667 -> 7 (control), wired pin share 0 -> 0.90 / 0.76, junctions,
hierarchical labels and power symbols introduced, continuation sheets removed; readability metrics
V2 vs V2.1 in engineering_checks/schematic_readability_*.

Power board (octilinear simplification + tangent arcs on the V2 search; 8-direction search kept
opt-in after attempt A left 2 connections open): 0 unresolved, DRC 0/0/0 (20261012T090308Z-drc-8fd50803),
segments 4755 -> 2991 + 145 arcs, 90-degree bends 3609 -> 1121, stair runs 382 -> 124, length
5744.6 -> 5545.6 mm, vias 606 = V2, no net longer / more vias / narrower. Control board: 0 unresolved,
DRC 0/0/0 (20261012T084327Z-drc-7f07f983), segments 5995 -> 4262 + 261 arcs, 90-degree bends
4069 -> 1233, stair runs 435 -> 144, length 7055.2 -> 6700.7 mm, vias 798 = V2, 96 nets shorter,
0 longer. FOOTPRINT.SetDNP for DNP parts (schematic parity), beautify anchors bound to off-grid vias
by copper overlap (path_geometry.connected_by_overlap), In2.Cu inner pass styled.

Exports 11/11 per board, renders and layer PDFs refreshed, high-resolution V2/V2.1 crops under
review/crops/, routing_quality_* and v21_validation.{json,md} (nine TASK 7 checks independently
re-derived). verify_sic_buck passed; 338 tests OK (2 skipped).

Co-Authored-By: Claude Fable 5.1 <noreply@anthropic.com>
Parts:
- added C34: 330p/50V, Capacitor_SMD:C_0603_1608Metric, symbol AIPE:Sym_C34
- added C35: 330p/50V, Capacitor_SMD:C_0603_1608Metric, symbol AIPE:Sym_C35
- added C36: 4.7u/25V, Capacitor_SMD:C_1206_3216Metric, symbol AIPE:Sym_C36
- added C37: 4.7u/25V, Capacitor_SMD:C_1206_3216Metric, symbol AIPE:Sym_C37
- added C38: 100n/50V, Capacitor_SMD:C_0603_1608Metric, symbol AIPE:Sym_C38
- added C39: 4.7u/25V, Capacitor_SMD:C_1206_3216Metric, symbol AIPE:Sym_C39
- added R29: 107k, Resistor_SMD:R_0603_1608Metric, symbol AIPE:Sym_R29
- added R30: 16.2k, Resistor_SMD:R_0603_1608Metric, symbol AIPE:Sym_R30
- added R31: 9.76k, Resistor_SMD:R_0603_1608Metric, symbol AIPE:Sym_R31
- added R32: 16.2k, Resistor_SMD:R_0603_1608Metric, symbol AIPE:Sym_R32
- added R33: 1k, Resistor_SMD:R_0805_2012Metric, symbol AIPE:Sym_R33
- added R34: 10k, Resistor_SMD:R_0603_1608Metric, symbol AIPE:Sym_R34
- added U2: UCC14141QDWNRQ1, AIPE:UCC14141_DWN0036A_Slot, symbol AIPE:Sym_U2
- C21, D4, R23: now not fitted
Connections:
- net 12V_BIAS_H: now also U2.6 (VIN), U2.7 (VIN)
- net 3V3: now also R34.1
- net GNDP_H: now also U2.1 (GNDP), U2.10 (GNDP), U2.11 (GNDP), U2.12 (GNDP), U2.13 (GNDP), U2.14 (GNDP), U2.15 (GNDP), U2.16 (GNDP), U2.17 (GNDP), U2.18 (GNDP), U2.2 (GNDP), U2.5 (GNDP), U2.8 (GNDP), U2.9 (GNDP)
- net KS_H: now also C39.1, R31.1, R33.2
- net VDD_H: now also C36.1, C37.1, C38.1, R29.1, U2.28 (VDD), U2.29 (VDD)
- net VEE_H: now also C34.2, C35.2, C36.2, C37.2, C38.2, C39.2, R30.2, R32.2, U2.19 (VEE), U2.20 (VEE), U2.21 (VEE), U2.22 (VEE), U2.23 (VEE), U2.24 (VEE), U2.25 (VEE), U2.26 (VEE), U2.27 (VEE), U2.30 (VEE), U2.31 (VEE), U2.35 (VEEA), U2.36 (VEE)
- new net BIAS_EN_F: U2.4 (ENA)
- new net HS_FB_VDD: C34.1, R29.2, R30.1, U2.34 (FBVDD)
- new net HS_FB_VEE: C35.1, R31.2, R32.1, U2.33 (FBVEE)
- new net HS_RLIM: R33.1, U2.32 (RLIM)
- new net PG_BIAS_H_N: R34.2, U2.3 (PG)
Other:
- note added: "HS DESAT protection network"
- note added: "HS isolated bias supply (UCC14141-Q1)"
- note added: "HS isolated gate driver (UCC21710-Q1): PWM input, gate network, status pull-ups, decoupling"
- note added: "Supply provenance (PWR_FLAG)"
- moved on the sheet: D3, L2, R23, TP1, U1
