File: examples/sic-buck-400v-200v-5kw/kicad/power_board/02_gate_driver_hs.kicad_sch (KiCad schematic)
At the start: 44 parts, among them U1 UCC21710QDWRQ1, U2 UCC14141QDWNRQ1

Commit message: Correct sensing circuits and add verified V2.2 local bypasses
Other:
- moved on the sheet: C20, C21, C22, C23, C24, C25, C26, C27, C28, C29, C30, C31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
