File: examples/sic-buck-400v-200v-5kw/kicad/power_board/03_gate_driver_ls.kicad_sch (KiCad schematic)
At the start: 31 parts, among them U3 UCC21710QDWRQ1

Commit message: fix(pcb): structural DRC sources removed at the schematic level; layout review and stage-3 evidence
Power project regenerated (ERC 0 findings, run 20261010T165532Z): UCC21710 drivers now use
an AIPE footprint that carries its own 1.2 x 16.6 mm isolation slot (no library
silkscreen crossing a board cut-out), the AMC1311 slot is lengthened to 10.8 mm, the
LED anode nodes of the indicator strings form a PGND_LV class of the PGND reference
island (0.3 mm to PGND instead of a 3 mm HV spacing an 0805 LED cannot meet), and the
pin-field exceptions now cover no-connect pads whose unconnected-* nets fall into
KiCad's Default class. 45 design rules; nothing weakened.

Also records the independent layout review of the first routed state
(pcb_rule_review.md, 19 findings), the correction pass before/after tables, the
stage-3 power-board routing experiments and patch set, the stage-1 floorplan
generator with its candidate comparison, run_check report hashes and the verifier
hash fix.

Co-Authored-By: Claude Fable 5.1 <noreply@anthropic.com>
Parts:
- U3: footprint Package_SO:SOIC-16W_7.5x10.3mm_P1.27mm -> AIPE:UCC21710_DW0016A_Slot
Changed lines of the file:
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@@
           (property "Reference" "U3" (at 240.03 34.29 0)  (effects (font (size 1.27 1.27))))
 (property "Value" "UCC21710QDWRQ1" (at 240.03 36.83 0)  (effects (font (size 1.27 1.27))))
-(property "Footprint" "Package_SO:SOIC-16W_7.5x10.3mm_P1.27mm" (at 240.03 52.07 0) (hide yes) (effects (font (size 1.27 1.27))))
+(property "Footprint" "AIPE:UCC21710_DW0016A_Slot" (at 240.03 52.07 0) (hide yes) (effects (font (size 1.27 1.27))))
 (property "Datasheet" "" (at 240.03 52.07 0) (hide yes) (effects (font (size 1.27 1.27))))
           (pin "1")

Commit message: feat(v2.1): example regenerated - wired schematics, both boards routed with the upgraded router, exports, crops, validation
Schematics (wired style, gates passed): ERC 0 on both projects (power 20261012T075113Z-erc-df18ce6e,
control 20261012T075120Z-erc-7a14cacb); netlist (ref,pad)->net exact vs the model and vs the frozen V2
netlists with equal net names; .kicad_dru / net_settings identical to the legacy generation; stub
global labels 648 -> 7 (power) and 667 -> 7 (control), wired pin share 0 -> 0.90 / 0.76, junctions,
hierarchical labels and power symbols introduced, continuation sheets removed; readability metrics
V2 vs V2.1 in engineering_checks/schematic_readability_*.

Power board (octilinear simplification + tangent arcs on the V2 search; 8-direction search kept
opt-in after attempt A left 2 connections open): 0 unresolved, DRC 0/0/0 (20261012T090308Z-drc-8fd50803),
segments 4755 -> 2991 + 145 arcs, 90-degree bends 3609 -> 1121, stair runs 382 -> 124, length
5744.6 -> 5545.6 mm, vias 606 = V2, no net longer / more vias / narrower. Control board: 0 unresolved,
DRC 0/0/0 (20261012T084327Z-drc-7f07f983), segments 5995 -> 4262 + 261 arcs, 90-degree bends
4069 -> 1233, stair runs 435 -> 144, length 7055.2 -> 6700.7 mm, vias 798 = V2, 96 nets shorter,
0 longer. FOOTPRINT.SetDNP for DNP parts (schematic parity), beautify anchors bound to off-grid vias
by copper overlap (path_geometry.connected_by_overlap), In2.Cu inner pass styled.

Exports 11/11 per board, renders and layer PDFs refreshed, high-resolution V2/V2.1 crops under
review/crops/, routing_quality_* and v21_validation.{json,md} (nine TASK 7 checks independently
re-derived). verify_sic_buck passed; 338 tests OK (2 skipped).

Co-Authored-By: Claude Fable 5.1 <noreply@anthropic.com>
Parts:
- added C54: 330p/50V, Capacitor_SMD:C_0603_1608Metric, symbol AIPE:Sym_C54
- added C55: 330p/50V, Capacitor_SMD:C_0603_1608Metric, symbol AIPE:Sym_C55
- added C56: 4.7u/25V, Capacitor_SMD:C_1206_3216Metric, symbol AIPE:Sym_C56
- added C57: 4.7u/25V, Capacitor_SMD:C_1206_3216Metric, symbol AIPE:Sym_C57
- added C58: 100n/50V, Capacitor_SMD:C_0603_1608Metric, symbol AIPE:Sym_C58
- added C59: 4.7u/25V, Capacitor_SMD:C_1206_3216Metric, symbol AIPE:Sym_C59
- added R47: 107k, Resistor_SMD:R_0603_1608Metric, symbol AIPE:Sym_R47
- added R48: 16.2k, Resistor_SMD:R_0603_1608Metric, symbol AIPE:Sym_R48
- added R49: 9.76k, Resistor_SMD:R_0603_1608Metric, symbol AIPE:Sym_R49
- added R50: 16.2k, Resistor_SMD:R_0603_1608Metric, symbol AIPE:Sym_R50
- added R51: 1k, Resistor_SMD:R_0805_2012Metric, symbol AIPE:Sym_R51
- added R52: 10k, Resistor_SMD:R_0603_1608Metric, symbol AIPE:Sym_R52
- added U4: UCC14141QDWNRQ1, AIPE:UCC14141_DWN0036A_Slot, symbol AIPE:Sym_U4
- C41, D6, R41: now not fitted
Connections:
- net 12V_BIAS_L: now also U4.6 (VIN), U4.7 (VIN)
- net 3V3: now also R52.1
- net GNDP_L: now also U4.1 (GNDP), U4.10 (GNDP), U4.11 (GNDP), U4.12 (GNDP), U4.13 (GNDP), U4.14 (GNDP), U4.15 (GNDP), U4.16 (GNDP), U4.17 (GNDP), U4.18 (GNDP), U4.2 (GNDP), U4.5 (GNDP), U4.8 (GNDP), U4.9 (GNDP)
- net KS_L: now also C59.1, R49.1, R51.2
- net VDD_L: now also C56.1, C57.1, C58.1, R47.1, U4.28 (VDD), U4.29 (VDD)
- net VEE_L: now also C54.2, C55.2, C56.2, C57.2, C58.2, C59.2, R48.2, R50.2, U4.19 (VEE), U4.20 (VEE), U4.21 (VEE), U4.22 (VEE), U4.23 (VEE), U4.24 (VEE), U4.25 (VEE), U4.26 (VEE), U4.27 (VEE), U4.30 (VEE), U4.31 (VEE), U4.35 (VEEA), U4.36 (VEE)
- new net BIAS_EN_F: U4.4 (ENA)
- new net LS_FB_VDD: C54.1, R47.2, R48.1, U4.34 (FBVDD)
- new net LS_FB_VEE: C55.1, R49.2, R50.1, U4.33 (FBVEE)
- new net LS_RLIM: R51.1, U4.32 (RLIM)
- new net PG_BIAS_L_N: R52.2, U4.3 (PG)
Other:
- note added: "LS DESAT protection network"
- note added: "LS isolated bias supply (UCC14141-Q1)"
- note added: "LS isolated gate driver (UCC21710-Q1): PWM input, gate network, status pull-ups, decoupling"
- note added: "Supply provenance (PWR_FLAG)"
- moved on the sheet: D5, L3, R41, TP2, U3
