File: examples/sic-buck-400v-200v-5kw/kicad/power_board/03_gate_driver_ls.kicad_sch (KiCad schematic)
At the start: 44 parts, among them U3 UCC21710QDWRQ1, U4 UCC14141QDWNRQ1

Commit message: Correct sensing circuits and add verified V2.2 local bypasses
Other:
- moved on the sheet: C40, C41, C42, C43, C44, C45, C46, C47, C48, C49, C50, C51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
