File: examples/sic-buck-400v-200v-5kw/kicad/power_board/04_sensing_island.kicad_sch (KiCad schematic)
At the start: 36 parts, among them U5 UCC14141QDWNRQ1, U6 AMC1311BDWVR, U7 AMC1311BDWVR

Commit message: Correct sensing circuits and add verified V2.2 local bypasses
Parts:
- R57: value 1k -> 160; footprint Resistor_SMD:R_0805_2012Metric -> Resistor_SMD:R_1206_3216Metric
Other:
- moved on the sheet: C60, C61, C62, C63, C64, C65, C66, C67, C68, C69, C70, C71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
