File: examples/sic-buck-400v-200v-5kw/kicad/power_board/05_selv_strip.kicad_sch (KiCad schematic)
At the start: 26 parts, among them J7 Mezzanine 2x25 socket, U8 OPA2320AIDGKR, U9 REF3125AIDBZR

Commit message: feat(v2.1): example regenerated - wired schematics, both boards routed with the upgraded router, exports, crops, validation
Schematics (wired style, gates passed): ERC 0 on both projects (power 20261012T075113Z-erc-df18ce6e,
control 20261012T075120Z-erc-7a14cacb); netlist (ref,pad)->net exact vs the model and vs the frozen V2
netlists with equal net names; .kicad_dru / net_settings identical to the legacy generation; stub
global labels 648 -> 7 (power) and 667 -> 7 (control), wired pin share 0 -> 0.90 / 0.76, junctions,
hierarchical labels and power symbols introduced, continuation sheets removed; readability metrics
V2 vs V2.1 in engineering_checks/schematic_readability_*.

Power board (octilinear simplification + tangent arcs on the V2 search; 8-direction search kept
opt-in after attempt A left 2 connections open): 0 unresolved, DRC 0/0/0 (20261012T090308Z-drc-8fd50803),
segments 4755 -> 2991 + 145 arcs, 90-degree bends 3609 -> 1121, stair runs 382 -> 124, length
5744.6 -> 5545.6 mm, vias 606 = V2, no net longer / more vias / narrower. Control board: 0 unresolved,
DRC 0/0/0 (20261012T084327Z-drc-7f07f983), segments 5995 -> 4262 + 261 arcs, 90-degree bends
4069 -> 1233, stair runs 435 -> 144, length 7055.2 -> 6700.7 mm, vias 798 = V2, 96 nets shorter,
0 longer. FOOTPRINT.SetDNP for DNP parts (schematic parity), beautify anchors bound to off-grid vias
by copper overlap (path_geometry.connected_by_overlap), In2.Cu inner pass styled.

Exports 11/11 per board, renders and layer PDFs refreshed, high-resolution V2/V2.1 crops under
review/crops/, routing_quality_* and v21_validation.{json,md} (nine TASK 7 checks independently
re-derived). verify_sic_buck passed; 338 tests OK (2 skipped).

Co-Authored-By: Claude Fable 5.1 <noreply@anthropic.com>
Parts:
- added C87: 100n/50V, Capacitor_SMD:C_0603_1608Metric, symbol AIPE:Sym_C87
- added C88: 1u/50V, Capacitor_SMD:C_0805_2012Metric, symbol AIPE:Sym_C88
- added C89: 100n/50V, Capacitor_SMD:C_0603_1608Metric, symbol AIPE:Sym_C89
- added C90: 100u/25V, Capacitor_SMD:CP_Elec_8x10.5, symbol AIPE:Sym_C90
- added C91: 10u/25V, Capacitor_SMD:C_1210_3225Metric, symbol AIPE:Sym_C91
- added D7: SS14 Schottky, Diode_SMD:D_SMA, symbol AIPE:Sym_D7
- added J8: FAN 12V/GND/TACH, Connector_PinHeader_2.54mm:PinHeader_1x03_P2.54mm_Vertical, symbol AIPE:Sym_J8
- added J9: Relay coil K1, TerminalBlock_Phoenix:TerminalBlock_Phoenix_MKDS-1,5-2-5.08_1x02_P5.08mm_Horizontal, symbol AIPE:Sym_J9
- added Q3: AO3400A, Package_TO_SOT_SMD:SOT-23, symbol AIPE:Sym_Q3
- added R81: 10k, Resistor_SMD:R_0603_1608Metric, symbol AIPE:Sym_R81
- added R82: 9.09k, Resistor_SMD:R_0603_1608Metric, symbol AIPE:Sym_R82
- added R83: 1k, Resistor_SMD:R_0603_1608Metric, symbol AIPE:Sym_R83
- added R84: 10k, Resistor_SMD:R_0603_1608Metric, symbol AIPE:Sym_R84
- added R85: 100, Resistor_SMD:R_0603_1608Metric, symbol AIPE:Sym_R85
- added R86: 10k, Resistor_SMD:R_0603_1608Metric, symbol AIPE:Sym_R86
Connections:
- net 12V_PROT: now also C90.1, C91.1, D7.1 (K), J8.1, J9.1
- net 3V3: now also C87.1, C88.1, R81.1, R82.1, R84.1
- net FAN_TACH: now also J8.3, R84.2
- net GND_CTRL: now also C87.2, C88.2, C89.2, C90.2, C91.2, J8.2, Q3.2 (S), R83.2, R86.2
- net ISENSE_REF: now also C89.1, R82.2, R83.1
- net OC_N: now also R81.2
- net RELAY_ON: now also R85.1
- new net K1_LOW: D7.2 (A), J9.2, Q3.3 (D)
- new net RLY_G: Q3.1 (G), R85.2, R86.1
Other:
- note added: "Mezzanine socket and receiving networks"
- note added: "OPA2320 difference amplifiers"
- note added: "REF3125 reference, OC threshold, ISENSE_REF"
- note added: "Relay coil drive, fan header, 12 V bulk"
- note added: "Supply provenance (PWR_FLAG)"
- moved on the sheet: J7, U8, U9
