File: examples/sic-buck-400v-200v-5kw/kicad/power_board/05_selv_strip.kicad_sch (KiCad schematic)
At the start: 41 parts, among them J7 Mezzanine 2x25 socket, J8 FAN 12V/GND/TACH, J9 Relay coil K1, Q3 AO3400A, U8 OPA2320AIDGKR, U9 REF3125AIDBZR

Commit message: Correct sensing circuits and add verified V2.2 local bypasses
Parts:
- R82: value 9.09k -> 6.65k
- R83: value 1k -> 1.01k
Connections:
- net 3V3: no longer R82.1
- net REF2V5_PB: now also R82.1
Other:
- moved on the sheet: C78, C79, C80, C81, C82, C83, C84, C85, C86, C87, C88, C89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
