File: examples/sic-buck-400v-200v-5kw/kicad/power_board/AIPE_SiC_Buck_Power.kicad_pcb (KiCad board)
At the start: 4 copper layers, 240 x 180 mm, 237 parts, among them J1 VIN_RAW (+IN), J2 PGND (-IN), J3 VOUT (+OUT), J4 PGND (-OUT), J5 RLY_A (VIN_RAW), J6 RLY_B (VIN), J7 Mezzanine 2x25 socket, J8 FAN 12V/GND/TACH, J9 Relay coil K1, Q1 C4MS025120K, Q2 C4MS025120K, Q3 AO3400A, U1 UCC21710QDWRQ1, U10 TMCS1133C2AQDVGR, U2 UCC14141QDWNRQ1, U3 UCC21710QDWRQ1, U4 UCC14141QDWNRQ1, U5 UCC14141QDWNRQ1, U6 AMC1311BDWVR, U7 AMC1311BDWVR, U8 OPA2320AIDGKR, U9 REF3125AIDBZR

Commit message: Correct sensing circuits and add verified V2.2 local bypasses
Parts:
- R57: value 1k -> 160; footprint Resistor_SMD:R_0805_2012Metric -> Resistor_SMD:R_1206_3216Metric
- R82: value 9.09k -> 6.65k
- R83: value 1k -> 1.01k
- moved R57 4.97 mm to (169.0, 137.2), turned to 0 degrees
Connections:
- R82 pad 1: 3V3 -> REF2V5_PB
Routing:
- net REF2V5_PB: track 12.4 -> 59.3 mm, vias 0 -> 2
- net 5V_ISO: track 63.6 -> 68.8 mm, vias 7 -> 6
- net 3V3: track 417.8 -> 413.2 mm, vias 22 -> 21
- net ISO_RLIM: track 8.15 -> 9.77 mm
Other:
- board text added: "AI-GENERATED ENGINEERING PROTOTYPE - V2.2 - HUMAN REVIEW REQUIRED"
- board text added: "AIPE SiC BUCK 400V -> 200V / 5kW - POWER BOARD V2.2"
- board text removed: "AI-GENERATED ENGINEERING PROTOTYPE - V2.1 - HUMAN REVIEW REQUIRED"
- board text removed: "AIPE SiC BUCK 400V -> 200V / 5kW - POWER BOARD V2.1"
