File: examples/sic-buck-400v-200v-5kw-v3/kicad/control_board/05_analog.kicad_sch (KiCad schematic)
At the start: 74 parts, among them J5 LEM HO 50-S-0100, U6 OPA4192IPWR, U7 REF3130AIDBZR, U8 OPA2320AIDGKR, U9 LM61CIM3/NOPB

Commit message: Design independent V3 floorplans and thermal fixture with native spacing checks
Parts:
- U8: footprint Package_SO:VSSOP-8_3x3mm_P0.65mm -> AIPE:V3_DGK8
Changed lines of the file:
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@@
           (property "Reference" "U8" (at 176.53 237.49 0)  (effects (font (size 1.27 1.27))))
 (property "Value" "OPA2320AIDGKR" (at 176.53 240.03 0)  (effects (font (size 1.27 1.27))))
-(property "Footprint" "Package_SO:VSSOP-8_3x3mm_P0.65mm" (at 176.53 251.46 0) (hide yes) (effects (font (size 1.27 1.27))))
+(property "Footprint" "AIPE:V3_DGK8" (at 176.53 251.46 0) (hide yes) (effects (font (size 1.27 1.27))))
 (property "Datasheet" "" (at 176.53 251.46 0) (hide yes) (effects (font (size 1.27 1.27))))
           (pin "3")
@@
           (property "Reference" "U8" (at 97.79 309.88 0)  (effects (font (size 1.27 1.27))))
 (property "Value" "OPA2320AIDGKR" (at 97.79 312.42 0)  (effects (font (size 1.27 1.27))))
-(property "Footprint" "Package_SO:VSSOP-8_3x3mm_P0.65mm" (at 97.79 323.85 0) (hide yes) (effects (font (size 1.27 1.27))))
+(property "Footprint" "AIPE:V3_DGK8" (at 97.79 323.85 0) (hide yes) (effects (font (size 1.27 1.27))))
 (property "Datasheet" "" (at 97.79 323.85 0) (hide yes) (effects (font (size 1.27 1.27))))
           (pin "5")
@@
           (property "Reference" "U8" (at 162.56 309.88 0)  (effects (font (size 1.27 1.27))))
 (property "Value" "OPA2320AIDGKR" (at 162.56 312.41999999999996 0)  (effects (font (size 1.27 1.27))))
-(property "Footprint" "Package_SO:VSSOP-8_3x3mm_P0.65mm" (at 162.56 322.58 0) (hide yes) (effects (font (size 1.27 1.27))))
+(property "Footprint" "AIPE:V3_DGK8" (at 162.56 322.58 0) (hide yes) (effects (font (size 1.27 1.27))))
 (property "Datasheet" "" (at 162.56 322.58 0) (hide yes) (effects (font (size 1.27 1.27))))
           (pin "4")
