File: examples/sic-buck-400v-200v-5kw-v3/kicad/control_board/06_trip.kicad_sch (KiCad schematic)
At the start: 57 parts, among them U10 TLV3202AIDGKR, U11 TLV3202AIDGKR, U12 TLV3202AIDGKR, U13 SN74LV04APWR, U14 SN74LV21APWR, U15 SN74LV21APWR, U16 SN74LV21APWR, U17 SN74LVC2G08DCTR, U18 SN74LVC1G74DCTR, U19 SN74LVC2G08DCTR

Commit message: Design independent V3 floorplans and thermal fixture with native spacing checks
Parts:
- U10, U11, U12: footprint Package_SO:VSSOP-8_3x3mm_P0.65mm -> AIPE:V3_DGK8
Changed lines of the file:
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@@
           (property "Reference" "U10" (at 111.76 53.34 0)  (effects (font (size 1.27 1.27))))
 (property "Value" "TLV3202AIDGKR" (at 111.76 55.88 0)  (effects (font (size 1.27 1.27))))
-(property "Footprint" "Package_SO:VSSOP-8_3x3mm_P0.65mm" (at 111.76 67.31 0) (hide yes) (effects (font (size 1.27 1.27))))
+(property "Footprint" "AIPE:V3_DGK8" (at 111.76 67.31 0) (hide yes) (effects (font (size 1.27 1.27))))
 (property "Datasheet" "" (at 111.76 67.31 0) (hide yes) (effects (font (size 1.27 1.27))))
           (pin "3")
@@
           (property "Reference" "U10" (at 219.71 53.34 0)  (effects (font (size 1.27 1.27))))
 (property "Value" "TLV3202AIDGKR" (at 219.71 55.88 0)  (effects (font (size 1.27 1.27))))
-(property "Footprint" "Package_SO:VSSOP-8_3x3mm_P0.65mm" (at 219.71 67.31 0) (hide yes) (effects (font (size 1.27 1.27))))
+(property "Footprint" "AIPE:V3_DGK8" (at 219.71 67.31 0) (hide yes) (effects (font (size 1.27 1.27))))
 (property "Datasheet" "" (at 219.71 67.31 0) (hide yes) (effects (font (size 1.27 1.27))))
           (pin "5")
@@
           (property "Reference" "U10" (at 60.96 138.43 0)  (effects (font (size 1.27 1.27))))
 (property "Value" "TLV3202AIDGKR" (at 60.96 140.97 0)  (effects (font (size 1.27 1.27))))
-(property "Footprint" "Package_SO:VSSOP-8_3x3mm_P0.65mm" (at 60.96 151.13 0) (hide yes) (effects (font (size 1.27 1.27))))
+(property "Footprint" "AIPE:V3_DGK8" (at 60.96 151.13 0) (hide yes) (effects (font (size 1.27 1.27))))
 (property "Datasheet" "" (at 60.96 151.13 0) (hide yes) (effects (font (size 1.27 1.27))))
           (pin "4")
@@
           (property "Reference" "U11" (at 167.64 146.05 0)  (effects (font (size 1.27 1.27))))
 (property "Value" "TLV3202AIDGKR" (at 167.64 148.59 0)  (effects (font (size 1.27 1.27))))
-(property "Footprint" "Package_SO:VSSOP-8_3x3mm_P0.65mm" (at 167.64 160.02 0) (hide yes) (effects (font (size 1.27 1.27))))
+(property "Footprint" "AIPE:V3_DGK8" (at 167.64 160.02 0) (hide yes) (effects (font (size 1.27 1.27))))
 (property "Datasheet" "" (at 167.64 160.02 0) (hide yes) (effects (font (size 1.27 1.27))))
           (pin "3")
@@
           (property "Reference" "U11" (at 111.76 238.76 0)  (effects (font (size 1.27 1.27))))
 (property "Value" "TLV3202AIDGKR" (at 111.76 241.29999999999998 0)  (effects (font (size 1.27 1.27))))
-(property "Footprint" "Package_SO:VSSOP-8_3x3mm_P0.65mm" (at 111.76 252.73 0) (hide yes) (effects (font (size 1.27 1.27))))
+(property "Footprint" "AIPE:V3_DGK8" (at 111.76 252.73 0) (hide yes) (effects (font (size 1.27 1.27))))
 (property "Datasheet" "" (at 111.76 252.73 0) (hide yes) (effects (font (size 1.27 1.27))))
           (pin "5")
@@
           (property "Reference" "U11" (at 176.53 231.14000000000001 0)  (effects (font (size 1.27 1.27))))
 (property "Value" "TLV3202AIDGKR" (at 176.53 233.68 0)  (effects (font (size 1.27 1.27))))
-(property "Footprint" "Package_SO:VSSOP-8_3x3mm_P0.65mm" (at 176.53 243.84 0) (hide yes) (effects (font (size 1.27 1.27))))
+(property "Footprint" "AIPE:V3_DGK8" (at 176.53 243.84 0) (hide yes) (effects (font (size 1.27 1.27))))
 (property "Datasheet" "" (at 176.53 243.84 0) (hide yes) (effects (font (size 1.27 1.27))))
           (pin "4")
@@
           (property "Reference" "U12" (at 102.87 331.47 0)  (effects (font (size 1.27 1.27))))
 (property "Value" "TLV3202AIDGKR" (at 102.87 334.01 0)  (effects (font (size 1.27 1.27))))
-(property "Footprint" "Package_SO:VSSOP-8_3x3mm_P0.65mm" (at 102.87 345.44 0) (hide yes) (effects (font (size 1.27 1.27))))
+(property "Footprint" "AIPE:V3_DGK8" (at 102.87 345.44 0) (hide yes) (effects (font (size 1.27 1.27))))
 (property "Datasheet" "" (at 102.87 345.44 0) (hide yes) (effects (font (size 1.27 1.27))))
           (pin "3")
@@
           (property "Reference" "U12" (at 218.44 323.85 0)  (effects (font (size 1.27 1.27))))
 (property "Value" "TLV3202AIDGKR" (at 218.44 326.39 0)  (effects (font (size 1.27 1.27))))
-(property "Footprint" "Package_SO:VSSOP-8_3x3mm_P0.65mm" (at 218.44 337.82 0) (hide yes) (effects (font (size 1.27 1.27))))
+(property "Footprint" "AIPE:V3_DGK8" (at 218.44 337.82 0) (hide yes) (effects (font (size 1.27 1.27))))
 (property "Datasheet" "" (at 218.44 337.82 0) (hide yes) (effects (font (size 1.27 1.27))))
           (pin "5")
@@
           (property "Reference" "U12" (at 60.96 392.43 0)  (effects (font (size 1.27 1.27))))
 (property "Value" "TLV3202AIDGKR" (at 60.96 394.96999999999997 0)  (effects (font (size 1.27 1.27))))
-(property "Footprint" "Package_SO:VSSOP-8_3x3mm_P0.65mm" (at 60.96 405.13 0) (hide yes) (effects (font (size 1.27 1.27))))
+(property "Footprint" "AIPE:V3_DGK8" (at 60.96 405.13 0) (hide yes) (effects (font (size 1.27 1.27))))
 (property "Datasheet" "" (at 60.96 405.13 0) (hide yes) (effects (font (size 1.27 1.27))))
           (pin "4")
