File: examples/sic-buck-400v-200v-5kw-v3/kicad/control_board/sic-v3-control.kicad_pcb (KiCad board)
At the start: 4 copper layers, 160 x 120 mm, 266 parts, among them J1 12 V ELECTRONICS, J10 PRE AUX CONTACT, J11 Series NC90C sink thermostat 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, J12 12V fan; open-collector tach;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, J13 POWER / CONTROL — 40-way, J2 RESET input, J3 TI 14-pin JTAG; pin6 key, J4 3.3 V UART; external cable le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, J5 LEM HO 50-S-0100, J6 12 V COIL / FAN, J7 MAIN COIL, J8 PRE COIL, J9 MAIN AUX CONTACT, Q1 MMBT3904,215, Q2 IRLZ44NPBF, Q3 IRLZ44NPBF, U1 TPS26400PWPR, U10 TLV3202AIDGKR, U11 TLV3202AIDGKR, U12 TLV3202AIDGKR, U13 SN74LV04APWR, U14 SN74LV21APWR, U15 SN74LV21APWR, U16 SN74LV21APWR, U17 SN74LVC2G08DCTR, U18 SN74LVC1G74DCTR, U19 SN74LVC2G08DCTR, U2 TPS54302DDCR, U20 SN74AHCT125PWR, U3 TPS767D301PWPR, U4 TPS3808G01DBVR, U5 TMS320F28335PGFA, U6 OPA4192IPWR, U7 REF3130AIDBZR, U8 OPA2320AIDGKR, U9 LM61CIM3/NOPB, Y1 ASV-30.000MHZ-EJ-T

Commit message: Complete V3 control routing and add native copper connectivity repair tools
Parts:
- C2: moved to B.Cu
- moved R64 15.2 mm to (111.8, 54.5), turned to 0 degrees
- moved R62 14.5 mm to (106.5, 49.2), turned to -90 degrees
- moved R57 11.9 mm to (103.2, 57.2), turned to 180 degrees
- moved D10 11.8 mm to (102.8, 45.8), turned to 90 degrees
- moved D13 11.4 mm to (112.8, 56.8)
- moved D15 10.7 mm to (110.0, 46.8)
- moved D11 9.95 mm to (111.2, 62.2)
- moved D8 9.89 mm to (109.2, 59.5)
- moved D14 9.57 mm to (110.0, 49.5)
- moved D16 9.43 mm to (108.5, 44.0)
- moved D12 8.90 mm to (108.5, 68.5)
- moved C67 8.84 mm to (102.5, 64.5), turned to -90 degrees
- moved R59 8.60 mm to (106.8, 61.8), turned to 180 degrees
- moved R65 8.28 mm to (113.5, 59.0), turned to 0 degrees
- moved R58 7.83 mm to (103.2, 61.8), turned to 180 degrees
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Routing:
- net 3V3: track 0.00 -> 874.3 mm, vias 0 -> 113
- net 5V: track 0.00 -> 368.6 mm, vias 0 -> 43
- net GND_CTRL: track 0.00 -> 340.3 mm, vias 0 -> 216
- net 1V9: track 0.00 -> 246.8 mm, vias 0 -> 40
- net AUX_OK_N: track 0.00 -> 217.5 mm, vias 0 -> 11
- net 12V_E: track 0.00 -> 202.7 mm, vias 0 -> 6
- net THERM_OK: track 0.00 -> 198.7 mm, vias 0 -> 11
- net FLT_L_N: track 0.00 -> 170.9 mm, vias 0 -> 7
- net FAN_TACH: track 0.00 -> 166.9 mm, vias 0 -> 6
- net XRS_N: track 0.00 -> 164.2 mm, vias 0 -> 14
- net PG_L_N: track 0.00 -> 160.1 mm, vias 0 -> 9
- net RDY_L: track 0.00 -> 153.5 mm, vias 0 -> 6
- net PG_H_N: track 0.00 -> 138.7 mm, vias 0 -> 12
- net FLT_H_N: track 0.00 -> 128.3 mm, vias 0 -> 9
- net RDY_H: track 0.00 -> 126.7 mm, vias 0 -> 5
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- added copper zone on In2.Cu, net 1V9
- added copper zone on In2.Cu, net 3V3
- added copper zone on In1.Cu, net GND_CTRL
