File: examples/sic-buck-400v-200v-5kw-v3/kicad/power_board/05_ls_bias.kicad_sch (KiCad schematic)
At the start: 23 parts, among them U4 UCC14141QDWNRQ1

Commit message: Design independent V3 floorplans and thermal fixture with native spacing checks
Parts:
- NT2: now left out of the parts list
Changed lines of the file:
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@@
             (reference "R39") (unit 1)))))
 (symbol (lib_id "AIPE:Sym_NT2") (at 170.18 156.21 270)
-          (unit 1) (in_bom yes) (on_board yes) (dnp no)
+          (unit 1) (in_bom no) (on_board yes) (dnp no)
           (property "Reference" "NT2" (at 173.482 154.94 90)  (effects (font (size 1.27 1.27)) (justify left)))
 (property "Value" "VEEA STAR" (at 173.482 157.48 90)  (effects (font (size 1.27 1.27)) (justify left)))
