File: examples/sic-buck-400v-200v-5kw-v3/kicad/power_board/sic-v3-power.kicad_pcb (KiCad board)
At the start: 4 copper layers, 250 x 180 mm, 202 parts, among them J1 INPUT LINK +, J2 INPUT / OUTPUT RETURN, J3 SW TO CHOKE, J4 CHOKE RETURN / OUTPUT +, J5 OUTPUT RETURN, J6 RAW INPUT SENSE, J7 POWER / CONTROL — 40-way, Q1 C4MS025120K, Q2 C4MS025120K, U1 UCC21710QDWRQ1, U2 UCC21710QDWRQ1, U3 UCC14141QDWNRQ1, U4 UCC14141QDWNRQ1, U5 AMC1311BDWVR, U6 AMC1311BDWVR, U7 AMC1311BDWVR, U8 UCC14141QDWNRQ1

Commit message: Verify and freeze V3 power routing, system assembly and engineering review package
Parts:
- C16, C17, C18, C21, C22, C26, C30, C32, C33, C34, C42, C50, C54, C55, C62, C81, C94, R13, R28, R33, R40: moved to B.Cu
- moved C18 17.6 mm to (120.0, 19.5), turned to -90 degrees
- moved C29 16.4 mm to (148.0, 3.75)
- moved C17 14.7 mm to (119.6, 22.6)
- moved R18 14.6 mm to (112.0, 20.2), turned to 90 degrees
- moved C32 13.2 mm to (148.2, 3.25)
- moved C16 12.9 mm to (117.6, 19.4), turned to -90 degrees
- moved C26 12.9 mm to (114.8, 21.0)
- moved R33 12.0 mm to (83.5, 13.2), turned to 0 degrees
- moved C94 10.1 mm to (134.5, 100.2), turned to 180 degrees
- moved C30 8.66 mm to (141.5, 12.0), turned to -90 degrees
- moved R13 8.60 mm to (118.2, 13.5), turned to 180 degrees
- moved R28 7.32 mm to (138.2, 2.50)
- moved C55 6.18 mm to (166.5, 18.8)
- moved C62 6.01 mm to (175.8, 20.5), turned to 180 degrees
- moved C50 5.55 mm to (81.2, 17.5), turned to 0 degrees
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Routing:
- net GND_CTRL: track 0.00 -> 395.7 mm, vias 0 -> 18
- net 3V3: track 0.00 -> 341.9 mm, vias 0 -> 19
- net BIAS_EN_F: track 0.00 -> 269.6 mm, vias 0 -> 10
- net KS_H: track 0.00 -> 243.7 mm, vias 0 -> 13
- net 12V_E: track 0.00 -> 224.8 mm, vias 0 -> 4
- net VDD_L: track 0.00 -> 198.7 mm, vias 0 -> 12
- net KS_L: track 0.00 -> 166.7 mm, vias 0 -> 13
- net DRV_RESET_F: track 0.00 -> 156.6 mm, vias 0 -> 4
- net VDD_H: track 0.00 -> 105.6 mm, vias 0 -> 11
- net VEE_H: track 0.00 -> 104.2 mm, vias 0 -> 22
- net S_5V: track 0.00 -> 103.6 mm, vias 0 -> 10
- net PWM_H_F: track 0.00 -> 103.2 mm, vias 0 -> 5
- net PWM_L_F: track 0.00 -> 101.3 mm, vias 0 -> 2
- net PG_L_N: track 0.00 -> 100.2 mm, vias 0 -> 4
- net PG_H_N: track 0.00 -> 97.3 mm, vias 0 -> 2
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- added copper zone on B.Cu, net BUS
- added copper zone on F.Cu, net BUS
- added copper zone on In2.Cu, net BUS
- added copper zone on B.Cu, net GNDP_H
- added copper zone on F.Cu, net GNDP_H
- added copper zone on B.Cu, net GNDP_L
- added copper zone on F.Cu, net GNDP_L
- added copper zone on B.Cu, net GNDP_S
- added copper zone on F.Cu, net GNDP_S
- added copper zone on In1.Cu, net GND_CTRL
- added copper zone on B.Cu, net PGND
- added copper zone on F.Cu, net PGND
- added copper zone on In1.Cu, net PGND
- added copper zone on In2.Cu, net PGND
- added copper zone on B.Cu, net RAW
- added copper zone on F.Cu, net RAW
- added copper zone on B.Cu, net SW
- added copper zone on F.Cu, net SW
- added copper zone on In1.Cu, net SW
- added copper zone on In2.Cu, net SW
- added copper zone on B.Cu, net VEE_H
- added copper zone on F.Cu, net VEE_H
- added copper zone on B.Cu, net VEE_L
- added copper zone on F.Cu, net VEE_L
- added copper zone on B.Cu, net VOUT
- added copper zone on F.Cu, net VOUT
- added copper zone on In1.Cu, net VOUT
- added copper zone on In2.Cu, net VOUT
