File: examples/dab-10kw/primary-power/dab-primary.kicad_pcb (KiCad board)
At the start: 4 copper layers, 300 x 150 mm, 309 parts, among them J1 DC BUS +, J2 DC BUS -, J3 AC A (switch node A), J4 AC B (transformer, via curren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, J5 CONTROL HARNESS 40-way, J6 HEATSINK NTC, Q1 C3M0075120K, Q2 C3M0075120K, Q3 C3M0075120K, Q4 C3M0075120K, U1 TMCS1133B1QDVGR, U10 UCC14141QDWNRQ1, U11 AMC1311BDWVR, U2 UCC21710QDWRQ1, U3 UCC14141QDWNRQ1, U4 UCC21710QDWRQ1, U5 UCC14141QDWNRQ1, U6 UCC21710QDWRQ1, U7 UCC14141QDWNRQ1, U8 UCC21710QDWRQ1, U9 UCC14141QDWNRQ1

Commit message: Remediate DAB-V1 routing: fine-pitch row escapes, exit lanes, plane continuity, time-boxed router
Root causes of the 2026-10-21 DRC failures and open connections of the three DAB-V1 boards are documented in
docs/dab-10kw/routing-remediation.md; the generator and the grid router were changed accordingly and the boards were
regenerated and re-verified with kicad-cli 10.0.6 (ERC, DRC --schematic-parity --severity-all --refill-zones, exports,
netlist equality, copper islands, barrier geometry).

Results (before -> after): primary 22 DRC errors -> 0, 82 unconnected -> 26; secondary 2 -> 0, 81 -> 23;
control not routed (499) -> routed, 0 errors, 24 unconnected. ERC 0 and parity 0 on all boards. Open connections
remain, so no board is manufacturing-ready.

Generator: fine-pitch row escapes (automation/dab_v1/fanout_rows.py: same-net bridges, one stub per run, computed stub
lengths, exit lanes), placement fan-out band and part gap, DESAT diode out of the plane band, sense pours joined to
the planes, AC_B riser over J4 capped at the Hall bars, 0.5 mm module input rails. Router: footprint copper graphics
as via exclusions, geometric stub-end acceptance, exit lanes at stub width (critical pads included), stranded ground
routing, time_budget_s with checkpoints. Tests added; KiCad-dependent tests gated for CI; pyproject 0.1.0; README in
the AIPE template (former README moved to docs/history.md).

Co-Authored-By: Claude Fable 5.1 <noreply@anthropic.com>
Parts:
- moved R46 16.6 mm to (151.0, 56.2), turned to -90 degrees
- moved R28 15.7 mm to (129.0, 48.5), turned to 180 degrees
- moved R62 15.5 mm to (189.8, 47.2), turned to 0 degrees
- moved C94 15.5 mm to (203.0, 50.0), turned to 180 degrees
- moved R29 14.9 mm to (115.0, 52.5), turned to 90 degrees
- moved C29 14.8 mm to (79.0, 56.2), turned to -90 degrees
- moved C53 14.8 mm to (115.0, 56.2), turned to -90 degrees
- moved C116 14.6 mm to (245.0, 85.5), turned to 180 degrees
- moved C101 14.6 mm to (187.0, 54.8), turned to -90 degrees
- moved C117 14.3 mm to (232.5, 89.0), turned to 180 degrees
- moved TP1 13.4 mm to (90.5, 59.0), turned to 180 degrees
- moved TP2 13.4 mm to (126.5, 59.0), turned to 180 degrees
- moved TP3 13.4 mm to (162.5, 59.0), turned to 180 degrees
- moved C35 13.1 mm to (100.2, 53.8), turned to 180 degrees
- moved C59 13.1 mm to (136.2, 53.8), turned to 180 degrees
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Routing:
- net PG_BIAS_N: track 47.3 -> 201.1 mm, vias 1 -> 7
- net DRV_RSTF: track 126.7 -> 261.6 mm
- net VSNS_P: track 0.90 -> 100.5 mm, vias 0 -> 1
- net VEE_BL: track 112.9 -> 182.4 mm, vias 6 -> 4
- net 3V3: track 412.7 -> 482.1 mm, vias 22 -> 31
- net SDFM_D: track 0.00 -> 59.1 mm, vias 0 -> 1
- net NTC_BL: track 24.5 -> 71.6 mm
- net VDD_AH: track 73.9 -> 120.5 mm, vias 13 -> 4
- net GNDP_S: track 87.5 -> 44.0 mm
- net VEE_AH: track 106.7 -> 71.6 mm, vias 7 -> 8
- net RLIM_AL: track 2.75 -> 31.8 mm, vias 0 -> 6
- net S_FBVDD: track 10.8 -> 37.9 mm
- net VEEA_AH: track 42.0 -> 16.7 mm
- net S_FBVEE: track 3.75 -> 28.0 mm, vias 0 -> 2
- net NTC_BH: track 24.5 -> 46.7 mm, vias 4 -> 5
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