File: examples/dab-10kw/secondary-power/dab-secondary.kicad_pcb (KiCad board)
At the start: 4 copper layers, 300 x 150 mm, 312 parts, among them J1 DC BUS +, J2 DC BUS -, J3 AC A (switch node A), J4 AC B (transformer, via curren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, J5 CONTROL HARNESS 40-way, J6 HEATSINK NTC, Q1 C3M0030090K, Q2 C3M0030090K, Q3 C3M0030090K, Q4 C3M0030090K, U1 TMCS1133B1QDVGR, U10 UCC14141QDWNRQ1, U11 AMC1311BDWVR, U12 AMC1336DWVR, U2 UCC21710QDWRQ1, U3 UCC14141QDWNRQ1, U4 UCC21710QDWRQ1, U5 UCC14141QDWNRQ1, U6 UCC21710QDWRQ1, U7 UCC14141QDWNRQ1, U8 UCC21710QDWRQ1, U9 UCC14141QDWNRQ1

Commit message: Remediate DAB-V1 routing: fine-pitch row escapes, exit lanes, plane continuity, time-boxed router
Root causes of the 2026-10-21 DRC failures and open connections of the three DAB-V1 boards are documented in
docs/dab-10kw/routing-remediation.md; the generator and the grid router were changed accordingly and the boards were
regenerated and re-verified with kicad-cli 10.0.6 (ERC, DRC --schematic-parity --severity-all --refill-zones, exports,
netlist equality, copper islands, barrier geometry).

Results (before -> after): primary 22 DRC errors -> 0, 82 unconnected -> 26; secondary 2 -> 0, 81 -> 23;
control not routed (499) -> routed, 0 errors, 24 unconnected. ERC 0 and parity 0 on all boards. Open connections
remain, so no board is manufacturing-ready.

Generator: fine-pitch row escapes (automation/dab_v1/fanout_rows.py: same-net bridges, one stub per run, computed stub
lengths, exit lanes), placement fan-out band and part gap, DESAT diode out of the plane band, sense pours joined to
the planes, AC_B riser over J4 capped at the Hall bars, 0.5 mm module input rails. Router: footprint copper graphics
as via exclusions, geometric stub-end acceptance, exit lanes at stub width (critical pads included), stranded ground
routing, time_budget_s with checkpoints. Tests added; KiCad-dependent tests gated for CI; pyproject 0.1.0; README in
the AIPE template (former README moved to docs/history.md).

Co-Authored-By: Claude Fable 5.1 <noreply@anthropic.com>
Parts:
- moved R68 17.7 mm to (199.0, 46.0), turned to 0 degrees
- moved R86 17.3 mm to (224.0, 44.8), turned to 180 degrees
- moved R44 16.6 mm to (151.0, 56.2), turned to -90 degrees
- moved C106 15.8 mm to (207.0, 51.2), turned to 0 degrees
- moved R26 15.7 mm to (129.0, 48.5), turned to 180 degrees
- moved C92 15.5 mm to (203.0, 50.0), turned to 180 degrees
- moved R27 14.9 mm to (115.0, 52.5), turned to 90 degrees
- moved C27 14.8 mm to (79.0, 56.2), turned to -90 degrees
- moved C51 14.8 mm to (115.0, 56.2), turned to -90 degrees
- moved C117 14.3 mm to (240.0, 50.2), turned to 180 degrees
- moved NT5 14.2 mm to (239.0, 52.5), turned to -90 degrees
- moved TP1 13.4 mm to (90.5, 59.0), turned to 180 degrees
- moved TP2 13.4 mm to (126.5, 59.0), turned to 180 degrees
- moved TP3 13.4 mm to (162.5, 59.0), turned to 180 degrees
- moved C33 13.1 mm to (100.2, 53.8), turned to 180 degrees
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Routing:
- net PG_BIAS_N: track 45.9 -> 260.0 mm, vias 1 -> 8
- net RDY_AL: track 74.1 -> 147.7 mm, vias 3 -> 1
- net VEE_BL: track 112.9 -> 182.4 mm, vias 6 -> 4
- net VDD_BH: track 117.8 -> 68.3 mm, vias 6 -> 3
- net 3V3: track 446.6 -> 494.1 mm, vias 23 -> 31
- net NTC_BL: track 24.5 -> 71.6 mm
- net VDD_AH: track 73.9 -> 120.5 mm, vias 13 -> 4
- net DRV_RSTF: track 118.4 -> 160.0 mm
- net VEE_AH: track 106.7 -> 71.6 mm, vias 7 -> 8
- net DESAT_BH: track 39.8 -> 5.97 mm
- net VMOD_IN: track 11.6 -> 45.4 mm
- net RLIM_AL: track 2.75 -> 31.8 mm, vias 0 -> 6
- net S_FBVDD: track 10.6 -> 38.7 mm, vias 3 -> 0
- net VEE_AL: track 109.7 -> 135.9 mm, vias 9 -> 6
- net VEEA_AH: track 42.0 -> 16.7 mm
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